File: tutorial/eagle/tutorial.brd (EAGLE design)
At the start: 99.1 x 73.7 mm, 16 parts, among them X2 8MHz, X4 MINI-USB

Commit message: update gerber to v1.6.1
Parts:
- added LED1, LED2, LED3: (no value), led:LED5MM
- added R2, R4, R5: (no value), rcl:R1206
- moved LDPW5 3.42 mm to (54.0, 42.5)
- moved R13 3.42 mm to (49.5, 42.5)
- moved C12 2.84 mm to (48.3, 54.6)
- moved C10 2.29 mm to (48.3, 51.4)
- moved R8 1.27 mm to (43.2, 39.4), turned to 180 degrees
Connections:
- new net N$5: LED3.K, R5.1
- new net N$6: LED2.K, R4.1
- new net N$7: LED1.K, R2.2
- net A0: now also LED1.A
- net A1: now also LED2.A
- net A2: now also LED3.A
- net GND: now also R2.1, R4.2, R5.2
Routing:
- net USB_P: track 0.00 -> 56.8 mm, vias 0 -> 2
- net USB_N: track 0.00 -> 56.6 mm, vias 0 -> 2
- net GND: track 0.00 -> 49.8 mm, vias 0 -> 5
- net RESET: track 0.00 -> 45.4 mm
- net MOSI: track 0.00 -> 36.5 mm
- net A2: track 0.00 -> 28.8 mm
- net VCC: track 0.00 -> 26.8 mm
- net A1: track 0.00 -> 23.9 mm
- net A0: track 0.00 -> 21.1 mm
- net N$42: track 0.00 -> 15.8 mm
- net XTAL1: track 0.00 -> 12.3 mm
- net USBC_N: track 0.00 -> 7.75 mm
- net USBC_P: track 0.00 -> 7.56 mm
- net N$7: track 0.00 -> 7.36 mm
- net N$6: track 0.00 -> 7.10 mm
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