File: hacking_the_simplespectro/pcb/eagle/main/hacking_the_simplespectro.brd (EAGLE design)
At the start: 99.1 x 73.7 mm, 56 parts, among them CON1 BAT, CON2 SPI, CON3 SPI, CON4 VIBR, IC1 32U4, IC2 MCP73831T, IC3 MCP1703CB, IC4 DMP1045U, Q6 BSP75, SW1 EC12E_SW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

Commit message: update eagle
Parts:
- removed LED5: RGB-COMMON-CATHODE, lpatiny:LED-TRICOLOR-THROUGHHOLE
- removed R8, R9: 1k, rcl:R0805
- added LED1: Blue, SparkFun:LED5MM
- R7: value 1k -> 22
- moved R7 3.86 mm to (64.1, 21.6)
Connections:
- removed net N$10: LED5.BLU, R8.1
- removed net N$9: LED5.GRN, R9.2
- net A0: no longer R7.2
- net A1: no longer R9.1
- net A2: now also R7.2; no longer R8.2
- net GND: now also LED1.A; no longer LED5.GND
- net N$13: now also LED1.K; no longer LED5.RED
Routing:
- net A0: track 55.5 -> 0.00 mm
- net A1: track 51.5 -> 0.00 mm
- net N$10: track 16.7 -> 0.00 mm
- net N$9: track 12.1 -> 0.00 mm
- net A2: track 47.5 -> 49.3 mm
Other:
- board text removed: "Green"
- board text removed: "Red"
Changed lines of the file:
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@@
 <text x="23.495" y="66.04" size="1.778" layer="52" rot="MR0">M</text>
 <text x="20.955" y="66.04" size="1.778" layer="52" rot="MR0">N</text>
-<text x="69.85" y="22.225" size="1.016" layer="52" rot="MR270">Red</text>
-<text x="66.675" y="22.86" size="1.016" layer="52" rot="MR270">Green</text>
 <text x="63.5" y="22.225" size="1.016" layer="52" rot="MR270">Blue</text>
 </plain>
@@
 <attribute name="VALUE" x="77.978" y="59.563" size="1.016" layer="28" ratio="10" rot="MR0"/>
 </element>
-<element name="R7" library="rcl" package="R0805" value="1k" x="67.945" y="20.955" smashed="yes" rot="MR90">
-<attribute name="ELECROW" value="C17513" x="67.945" y="20.955" size="1.778" layer="28" rot="MR90" display="off"/>
-<attribute name="LCSC" value="C17513" x="67.945" y="20.955" size="1.778" layer="28" rot="MR90" display="off"/>
-<attribute name="NAME" x="69.215" y="20.32" size="1.27" layer="26" rot="MR90"/>
-<attribute name="VALUE" x="67.31" y="23.495" size="1.27" layer="28" rot="MR90"/>
-</element>
-<element name="R8" library="rcl" package="R0805" value="1k" x="61.595" y="20.955" smashed="yes" rot="MR90">
-<attribute name="ELECROW" value="C17513" x="61.595" y="20.955" size="1.778" layer="28" rot="MR90" display="off"/>
-<attribute name="LCSC" value="C17513" x="61.595" y="20.955" size="1.778" layer="28" rot="MR90" display="off"/>
-<attribute name="NAME" x="62.865" y="20.32" size="1.27" layer="26" rot="MR90"/>
-<attribute name="VALUE" x="60.96" y="23.495" size="1.27" layer="28" rot="MR90"/>
-</element>
-<element name="R9" library="rcl" package="R0805" value="1k" x="64.77" y="20.955" smashed="yes" rot="MR270">
-<attribute name="ELECROW" value="C17513" x="64.77" y="20.955" size="1.778" layer="28" rot="MR270" display="off"/>
-<attribute name="LCSC" value="C17513" x="64.77" y="20.955" size="1.778" layer="28" rot="MR270" display="off"/>
-<attribute name="NAME" x="63.5" y="21.59" size="1.27" layer="26" rot="MR270"/>
-<attribute name="VALUE" x="65.41135" y="25.58415" size="1.27" layer="28" rot="MR270"/>
-</element>
-<element name="LED5" library="lpatiny" package="LED-TRICOLOR-THROUGHHOLE" value="RGB-COMMON-CATHODE" x="68.58" y="12.065" rot="MR270"/>
+<element name="R7" library="rcl" package="R0805" value="22" x="64.135" y="21.59" smashed="yes" rot="MR90">
+<attribute name="ELECROW" value="C17513" x="64.135" y="21.59" size="1.778" layer="28" rot="MR90" display="off"/>
+<attribute name="LCSC" value="C17513" x="64.135" y="21.59" size="1.778" layer="28" rot="MR90" display="off"/>
+<attribute name="NAME" x="65.405" y="20.955" size="1.27" layer="26" rot="MR90"/>
+<attribute name="VALUE" x="63.5" y="24.13" size="1.27" layer="28" rot="MR90"/>
+</element>
 <element name="LCD" library="HD44780LCD" package="LCD-16X2-4HOLES" value="LCD-HD447804-HOLES16X2-4-HOLES" x="49.53" y="53.34"/>
 <element name="C8" library="rcl" library_urn="urn:adsk.eagle:library:334" package="C0805K" package3d_urn="urn:adsk.eagle:package:23681/2" value="10u" x="69.85" y="41.91" smashed="yes" rot="MR0">
@@
 <attribute name="VALUE" x="80.4956" y="8.4801" size="1.27" layer="27" rot="R90"/>
 </element>
+<element name="LED1" library="SparkFun" package="LED5MM" value="Blue" x="64.135" y="13.335" rot="R90"/>
 </elements>
 <signals>
@@
 <wire x1="27.305" y1="38.8112" x2="27.0764" y2="39.0398" width="0.4064" layer="16"/>
 <via x="27.0764" y="39.0398" extent="1-16" drill="0.3048" shape="square"/>
-<contactref element="LED5" pad="GND"/>
 <wire x1="37.63" y1="37.97" x2="37.465" y2="37.97" width="0.4064" layer="16"/>
 <wire x1="37.465" y1="37.97" x2="37.465" y2="38.1" width="0.4064" layer="16"/>
@@
 <contactref element="SW1" pad="C"/>
 <contactref element="SW1" pad="E"/>
+<contactref element="LED1" pad="A"/>
+<wire x1="75.01214375" y1="66.04" x2="78.74" y2="69.85" width="0" layer="19" extent="16-16"/>
+<wire x1="72.025" y1="69.215" x2="72.39" y2="66.04" width="0" layer="19" extent="16-16"/>
+<wire x1="78.47" y1="55.245" x2="76.2" y2="61.595" width="0" layer="19" extent="16-16"/>
+<wire x1="83.82" y1="50.165" x2="78.74" y2="53.34" width="0" layer="19" extent="16-16"/>
+<wire x1="88.9" y1="41.58" x2="83.82" y2="49.26" width="0" layer="19" extent="16-16"/>
+<wire x1="83.82" y1="36.465" x2="88.265" y2="40.64" width="0" layer="19" extent="16-16"/>
+<wire x1="55.63" y1="68.84" x2="66.04" y2="67.945" width="0" layer="19" extent="1-1"/>
+<wire x1="51.435" y1="59.37" x2="55.63" y2="68.84" width="0" layer="19" extent="16-16"/>
+<wire x1="47.305" y1="54" x2="48.31" y2="59.37" width="0" layer="19" extent="16-16"/>
+<wire x1="42.63" y1="47.6" x2="42.63" y2="54" width="0" layer="19" extent="16-16"/>
+<wire x1="37.63" y1="45" x2="42.63" y2="47.6" width="0" layer="19" extent="16-16"/>
+<wire x1="42.545" y1="35.56" x2="37.63" y2="37.97" width="0" layer="19" extent="16-16"/>
+<wire x1="31.03" y1="49.2" x2="37.63" y2="45" width="0" layer="19" extent="16-16"/>
+<wire x1="32.83" y1="56.6" x2="31.03" y2="49.2" width="0" layer="19" extent="16-16"/>
+<wire x1="20.955" y1="55.88" x2="27.69" y2="59.0804" width="0" layer="19" extent="16-16"/>
+<wire x1="18.415" y1="47.26" x2="18.415" y2="55.61" width="0" layer="19" extent="16-16"/>
+<wire x1="27.305" y1="38.8112" x2="35.8775" y2="38.37" width="0" layer="19" extent="16-16"/>
+<wire x1="17.53" y1="68.84" x2="27.69" y2="68.84" width="0" layer="19" extent="1-1"/>
+<wire x1="8.255" y1="53.34" x2="18.415" y2="55.61" width="0" layer="19" extent="16-16"/>
+<wire x1="64.45" y1="44.915" x2="51.435" y2="46.0375" width="0" layer="19" extent="16-16"/>
+<wire x1="77.5506" y1="12.6151" x2="84.455" y2="34.925" width="0" layer="19" extent="16-16"/>
+<wire x1="92.0506" y1="10.1151" x2="77.5506" y2="12.6151" width="0" layer="19" extent="1-1"/>
+<wire x1="27.305" y1="14.097" x2="27.305" y2="37.465" width="0" layer="19" extent="16-16"/>
+<wire x1="32.725" y1="14.115" x2="27.305" y2="14.097" width="0" layer="19" extent="16-16"/>
+<wire x1="5.08" y1="13.335" x2="18.974" y2="2.769" width="0" layer="19" extent="16-16"/>
+<wire x1="64.135" y1="12.065" x2="18.974" y2="2.769" width="0" layer="19" extent="16-16"/>
 </signal>
 <signal name="SCK">
@@
 <wire x1="58.42" y1="50.965" x2="58.42" y2="25.7302" width="0.4064" layer="16"/>
 <wire x1="58.42" y1="25.7302" x2="59.055" y2="25.0952" width="0.4064" layer="16"/>
-<wire x1="59.055" y1="25.0952" x2="60.96" y2="25.0952" width="0.4064" layer="16"/>
 <wire x1="58.42" y1="50.965" x2="57.785" y2="51.6" width="0.4064" layer="16"/>
 <wire x1="57.785" y1="51.6" x2="42.63" y2="51.6" width="0.4064" layer="16"/>
-<contactref element="R8" pad="2"/>
-<wire x1="60.96" y1="25.0952" x2="61.595" y2="24.4602" width="0.4064" layer="16"/>
-<wire x1="61.595" y1="24.4602" x2="61.595" y2="21.905" width="0.4064" layer="16"/>
+<contactref element="R7" pad="2"/>
+<wire x1="63.1698" y1="25.0952" x2="64.135" y2="24.13" width="0.4064" layer="16"/>
+<wire x1="64.135" y1="24.13" x2="64.135" y2="22.54" width="0.4064" layer="16"/>
+<wire x1="59.055" y1="25.0952" x2="63.1698" y2="25.0952" width="0.4064" layer="16"/>
 </signal>
 <signal name="A3">
@@
 <signal name="A1">
 <contactref element="IC1" pad="37"/>
-<wire x1="59.4106" y1="51.765" x2="59.4106" y2="26.67" width="0.4064" layer="16"/>
-<wire x1="59.4106" y1="26.67" x2="60.0456" y2="26.035" width="0.4064" layer="16"/>
-<wire x1="60.0456" y1="26.035" x2="64.135" y2="26.035" width="0.4064" layer="16"/>
-<wire x1="59.4106" y1="51.765" x2="58.7756" y2="52.4" width="0.4064" layer="16"/>
-<wire x1="58.7756" y1="52.4" x2="42.63" y2="52.4" width="0.4064" layer="16"/>
-<contactref element="R9" pad="1"/>
-<wire x1="64.135" y1="26.035" x2="64.77" y2="25.4" width="0.4064" layer="16"/>
-<wire x1="64.77" y1="25.4" x2="64.77" y2="21.905" width="0.4064" layer="16"/>
 </signal>
 <signal name="D5">
@@
 <signal name="A0">
 <contactref element="IC1" pad="36"/>
-<contactref element="R7" pad="2"/>
-<wire x1="42.63" y1="53.2" x2="59.69" y2="53.2" width="0.4064" layer="16"/>
-<wire x1="59.69" y1="53.2" x2="60.325" y2="52.565" width="0.4064" layer="16"/>
-<wire x1="60.325" y1="52.565" x2="60.325" y2="27.6098" width="0.4064" layer="16"/>
-<wire x1="60.325" y1="27.6098" x2="60.96" y2="26.9748" width="0.4064" layer="16"/>
-<wire x1="60.96" y1="26.9748" x2="67.31" y2="26.9748" width="0.4064" layer="16"/>
-<wire x1="67.31" y1="26.9748" x2="67.945" y2="26.3398" width="0.4064" layer="16"/>
-<wire x1="67.945" y1="26.3398" x2="67.945" y2="21.905" width="0.4064" layer="16"/>
 </signal>
 <signal name="D12">
@@
 <wire x1="77.785" y1="64.1701" x2="77.785" y2="61.595" width="0.4064" layer="16"/>
 </signal>
-<signal name="N$9">
-<contactref element="LED5" pad="GRN"/>
-<contactref element="R9" pad="2"/>
-<wire x1="68.58" y1="11.319" x2="65.405" y2="11.319" width="0.4064" layer="16"/>
-<wire x1="65.405" y1="11.319" x2="64.77" y2="11.954" width="0.4064" layer="16"/>
-<wire x1="64.77" y1="11.954" x2="64.77" y2="20.005" width="0.4064" layer="16"/>
-</signal>
-<signal name="N$10">
-<contactref element="R8" pad="1"/>
-<contactref element="LED5" pad="BLU"/>
-<wire x1="68.58" y1="9.8905" x2="62.23" y2="9.8905" width="0.4064" layer="16"/>
-<wire x1="62.23" y1="9.8905" x2="61.595" y2="10.5255" width="0.4064" layer="16"/>
-<wire x1="61.595" y1="10.5255" x2="61.595" y2="20.005" width="0.4064" layer="16"/>
-</signal>
 <signal name="N$13">
-<contactref element="LED5" pad="RED"/>
 <contactref element="R7" pad="1"/>
-<wire x1="67.945" y1="20.005" x2="67.945" y2="14.811" width="0.4064" layer="16"/>
-<wire x1="67.945" y1="14.811" x2="68.58" y2="14.176" width="0.4064" layer="16"/>
+<contactref element="LED1" pad="K"/>
+<wire x1="64.135" y1="20.64" x2="64.135" y2="14.605" width="0.4064" layer="16"/>
 </signal>
 <signal name="VDD" class="1">
